File: pcb/intercons/intercons.kicad_pcb (KiCad board)
At the start: 2 copper layers, 76.4 x 84.6 mm, 16 parts, among them J1 COMM_OUT, J2 COMM_PSU, J3 COMM_BAT, J4 PSU, J5 BATTERY, J6 RoboClaw1, J7 RoboClaw2, J8 U2D2, SW1 PWR_SWITCH

Commit message: replaced wrong intercons pcb files
Parts:
- added logo1: LOGO, LOGO, B.Cu at (134.6, 63.4)
- added logo3: LOGO, LOGO, F.Cu at (150.6, 126.4)
- moved R1 23.4 mm to (159.8, 99.3)
- moved D2 7.20 mm to (134.1, 94.3)
- moved D1 7.18 mm to (134.0, 85.1)
- moved C1 4.77 mm to (120.7, 85.4)
- moved D3 4.02 mm to (159.8, 94.8)
- moved SW1 3.58 mm to (159.7, 85.1)
Routing:
- net GND: track 296.3 -> 0.00 mm
- net Net-(J1-Pin_1): track 59.7 -> 35.0 mm
- net Net-(D3-K): track 24.5 -> 4.54 mm
- net Net-(D2-A): track 143.4 -> 136.5 mm
- net Net-(A1-Bat+): track 99.7 -> 94.3 mm
- net Net-(A1-Vin+): track 34.8 -> 37.9 mm
- net Net-(A2-Vin+): track 63.8 -> 60.8 mm
- net Net-(D1-A): track 58.5 -> 57.5 mm
- added copper zone on B.Cu, net GND
- added copper zone on F.Cu, net GND
Other:
- board size 76.4 x 84.6 mm -> 77.8 x 84.6 mm
- board text added: "LARA Project Lucas Herrera UPM 2025"
- board text removed: "Lucas Herrera UPM 2025"
