File: pcb/LARA_hat/LARA_hat.kicad_pcb (KiCad board)
At the start: 2 copper layers, 65 x 56 mm, 30 parts, among them J1 Raspberry_Pi_4, J2 Conn_RoboClaw, J3 Conn_Dynamixel, J4 Conn_01x02_Pin, J5 12V in, J7 I2C_JST, U1 MCP2515-xSO, U2 SN65HVD230, U3 74LVC2G241, U4 Buck 12V - 5V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

Commit message: pcb
Routing:
- net GND: track 55.4 -> 68.7 mm, vias 3 -> 6
Changed lines of the file:
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@@
+	)
+	(segment
+		(start 136.8044 79.1956)
+		(end 137 79)
+		(width 0.2)
+		(layer "F.Cu")
+		(net 2)
 	)
 	(segment
@@
 	)
 	(segment
+		(start 160.401 110.3376)
+		(end 160.401 111.599)
+		(width 0.2)
+		(layer "F.Cu")
+		(net 2)
+	)
+	(segment
+		(start 163 113)
+		(end 163 113.9586)
+		(width 0.2)
+		(layer "F.Cu")
+		(net 2)
+	)
+	(segment
 		(start 141.1009 112.6744)
 		(end 139.1412 112.6744)
@@
 	)
 	(segment
+		(start 163 113.9586)
+		(end 161.671 115.2876)
+		(width 0.2)
+		(layer "F.Cu")
+		(net 2)
+	)
+	(segment
+		(start 160.401 111.599)
+		(end 160 112)
+		(width 0.2)
+		(layer "F.Cu")
+		(net 2)
+	)
+	(segment
+		(start 136.8044 81.1854)
+		(end 136.8044 79.1956)
+		(width 0.2)
+		(layer "F.Cu")
+		(net 2)
+	)
+	(segment
 		(start 142.4432 116.5524)
 		(end 143.3924 117.5016)
 		(width 0.2)
 		(layer "F.Cu")
+		(net 2)
+	)
+	(via
+		(at 137 79)
+		(size 0.6)
+		(drill 0.3)
+		(layers "F.Cu" "B.Cu")
 		(net 2)
 	)
@@
 		(net 2)
 	)
+	(via
+		(at 160 112)
+		(size 0.6)
+		(drill 0.3)
+		(layers "F.Cu" "B.Cu")
+		(net 2)
+	)
+	(via
+		(at 163 113)
+		(size 0.6)
+		(drill 0.3)
+		(layers "F.Cu" "B.Cu")
+		(net 2)
+	)
+	(segment
+		(start 137.0016 79)
+		(end 139.0904 76.9112)
+		(width 0.2)
+		(layer "B.Cu")
+		(net 2)
+	)
 	(segment
 		(start 152.8064 105.4608)
@@
 	)
 	(segment
+		(start 160 112)
+		(end 161 113)
+		(width 0.2)
+		(layer "B.Cu")
+		(net 2)
+	)
+	(segment
+		(start 137 79)
+		(end 137.0016 79)
+		(width 0.2)
+		(layer "B.Cu")
+		(net 2)
+	)
+	(segment
 		(start 139.0396 112.5728)
 		(end 142.4432 115.9764)
@@
 		(start 142.4432 115.9764)
 		(end 142.4432 116.5524)
+		(width 0.2)
+		(layer "B.Cu")
+		(net 2)
+	)
+	(segment
+		(start 161 113)
+		(end 163 113)
 		(width 0.2)
 		(layer "B.Cu")
@@
 		(layer "F.Cu")
 		(hatch edge 0.5)
-		(connect_pads
+		(connect_pads yes
 			(clearance 0.5)
 		)
@@
 		(hatch edge 0.5)
 		(priority 1)
-		(connect_pads
+		(connect_pads yes
 			(clearance 0.5)
 		)

Commit message: pcb
Parts:
- added J6: LED_JST, Connector_JST:JST_PH_B4B-PH-K_1x04_P2.00mm_Vertical, F.Cu at (137.0, 84.0)
- moved R10 15.8 mm to (149.0, 85.0), turned to -90 degrees
- moved R9 9.62 mm to (146.0, 85.0), turned to -90 degrees
- moved J2 6.41 mm to (137.0, 125.0), turned to 180 degrees
- moved J7 5.89 mm to (137.0, 116.0), turned to 180 degrees
- moved R8 4.07 mm to (143.0, 85.0), turned to -90 degrees
- moved C3 3.95 mm to (153.9, 112.7)
- moved C4 3.95 mm to (146.1, 112.8)
- moved R2 3.95 mm to (155.2, 120.0)
- moved R3 3.95 mm to (150.6, 120.0)
- moved R4 3.95 mm to (146.3, 120.0)
- moved U3 3.95 mm to (150.0, 116.0)
- moved U4 2.23 mm to (176.0, 100.0)
- moved R1 2.02 mm to (166.0, 81.0)
- moved D5 1.57 mm to (149.0, 81.0)
- moved J3 1.54 mm to (146.0, 124.0)
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Routing:
- net GND: track 68.7 -> 102.8 mm, vias 6 -> 9
- net +3V3: track 135.4 -> 103.0 mm, vias 4 -> 5
- net Net-(J1-GPCLK0/GPIO04): track 53.5 -> 73.9 mm
- net Net-(D5-A): track 7.44 -> 27.2 mm
- net Net-(J1-MISO_SPI0/GPIO09): track 29.6 -> 13.0 mm
- net Net-(D5-K): track 18.2 -> 1.97 mm
- net Net-(J1-GPCLK1/GPIO05): track 68.9 -> 56.1 mm
- net Net-(D4-A): track 7.76 -> 20.1 mm, vias 0 -> 1
- net +5V: track 75.2 -> 63.8 mm
- net Net-(J1-MOSI_SPI0/GPIO10): track 26.6 -> 16.0 mm
- net Net-(D4-K): track 10.6 -> 1.97 mm
- net Net-(J1-GPIO15/UART_RXD): track 75.7 -> 67.7 mm
- net Net-(D3-A): track 6.21 -> 12.6 mm
- net Net-(D2-A): track 42.4 -> 37.7 mm
- net Net-(J1-GPIO14/UART_TXD): track 68.2 -> 72.8 mm
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Other:
- outline, holes or cut-outs redrawn

Commit message: replaced wrong intercons pcb files
Parts:
- moved J3 0.86 mm to (145.9, 123.1)
- moved J2 0.81 mm to (137.1, 124.2)
- moved J5 0.77 mm to (171.2, 123.3)
- moved J4 0.67 mm to (161.7, 124.4)
- moved R3 0.32 mm to (150.9, 120.0)
- moved R4 0.24 mm to (146.1, 120.0)
Other:
- board text added: "12V IN"
- board text added: "CAN"
- board text added: "Dynamixel"
- board text added: "I2C"
- board text added: "RoboClaw"
Changed lines of the file:
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@@
 	(footprint "Connector_JST:JST_EH_B3B-EH-A_1x03_P2.50mm_Vertical"
 		(layer "F.Cu")
-		(at 146 124)
+		(at 145.9268 123.1392)
 		(descr "JST EH series connector, B3B-EH-A (http://www.jst-mfg.com/product/pdf/eng/eEH.pdf), generated with kicad-footprint-generator")
 		(tags "connector JST EH vertical")
@@
 		(tags "resistor handsolder")
 		(property "Reference" "R5"
-			(at 0 -1.65 0)
+			(at 0.1176 1.4224 0)
 			(layer "F.SilkS")
 			(effects
@@
 	(footprint "Connector_JST:JST_PH_B3B-PH-K_1x03_P2.00mm_Vertical"
 		(layer "F.Cu")
-		(at 137 125 180)
+		(at 137.0772 124.1972 180)
 		(descr "JST PH series connector, B3B-PH-K (http://www.jst-mfg.com/product/pdf/eng/ePH.pdf), generated with kicad-footprint-generator")
 		(tags "connector JST PH vertical")
@@
 	(footprint "Resistor_SMD:R_0805_2012Metric_Pad1.20x1.40mm_HandSolder"
 		(layer "F.Cu")
-		(at 150.6096 119.9722 180)
+		(at 150.9268 119.9722 180)
 		(descr "Resistor SMD 0805 (2012 Metric), square (rectangular) end terminal, IPC-7351 nominal with elongated pad for handsoldering. (Body size source: IPC-SM-782 page 72, https://www.pcb-3d.com/wordpress/wp-content/uploads/ipc-sm-782a_amendment_1_and_2.pdf), generated with kicad-footprint-generator")
 		(tags "resistor handsolder")
 		(property "Reference" "R3"
-			(at 0 -1.65 0)
+			(at -0.1016 1.5574 0)
 			(layer "F.SilkS")
 			(effects
@@
 	(footprint "TerminalBlock:TerminalBlock_MaiXu_MX126-5.0-02P_1x02_P5.00mm"
 		(layer "F.Cu")
-		(at 171.0436 124.0536)
+		(at 171.1744 123.2916)
 		(descr "terminal block MaiXu MX126-5.0-02P, 2 pins, pitch 5mm, size 10.5x7.8mm, drill diameter 1.3mm, pad diameter 2.8mm, https://www.lcsc.com/datasheet/lcsc_datasheet_2309150913_MAX-MX126-5-0-03P-GN01-Cu-S-A_C5188435.pdf, script-generated using https://gitlab.com/kicad/libraries/kicad-footprint-generator/-/tree/master/scripts/TerminalBlock_MaiXu")
 		(tags "THT terminal block MaiXu MX126-5.0-02P pitch 5mm size 10.5x7.8mm drill 1.3mm pad 2.8mm")
@@
 	(footprint "Resistor_SMD:R_0805_2012Metric_Pad1.20x1.40mm_HandSolder"
 		(layer "F.Cu")
-		(at 146.3424 119.9722)
+		(at 146.1008 119.9896)
 		(descr "Resistor SMD 0805 (2012 Metric), square (rectangular) end terminal, IPC-7351 nominal with elongated pad for handsoldering. (Body size source: IPC-SM-782 page 72, https://www.pcb-3d.com/wordpress/wp-content/uploads/ipc-sm-782a_amendment_1_and_2.pdf), generated with kicad-footprint-generator")
 		(tags "resistor handsolder")
@@
 	(footprint "Connector_JST:JST_PH_B2B-PH-K_1x02_P2.00mm_Vertical"
 		(layer "F.Cu")
-		(at 161.7472 125.0696 180)
+		(at 161.6804 124.4004 180)
 		(descr "JST PH series connector, B2B-PH-K (http://www.jst-mfg.com/product/pdf/eng/ePH.pdf), generated with kicad-footprint-generator")
 		(tags "connector JST PH vertical")
@@
 		(layer "Edge.Cuts")
 	)
+	(gr_text "12V IN"
+		(at 175.0568 118.2624 0)
+		(layer "F.SilkS")
+		(effects
+			(font
+				(size 1 1)
+				(thickness 0.1)
+			)
+			(justify left bottom)
+		)
+	)
+	(gr_text "CAN"
+		(at 159.0548 121.1072 0)
+		(layer "F.SilkS")
+		(effects
+			(font
+				(size 1 1)
+				(thickness 0.1)
+			)
+			(justify left bottom)
+		)
+	)
+	(gr_text "Dynamixel"
+		(at 144.6276 127.2032 0)
+		(layer "F.SilkS")
+		(effects
+			(font
+				(size 1 1)
+				(thickness 0.1)
+			)
+			(justify left bottom)
+		)
+	)
+	(gr_text "I2C"
+		(at 132.7912 112.3188 0)
+		(layer "F.SilkS")
+		(effects
+			(font
+				(size 1 1)
+				(thickness 0.1)
+			)
+			(justify left bottom)
+		)
+	)
+	(gr_text "RoboClaw"
+		(at 131.7244 120.8532 0)
+		(layer "F.SilkS")
+		(effects
+			(font
+				(size 1 1)
+				(thickness 0.1)
+			)
+			(justify left bottom)
+		)
+	)
 	(segment

Commit message: pcb gerbers
Parts:
- added G***: LOGO, LOGO, F.Cu at (124.9, 120.0)
- added G***: LOGO, LOGO, F.Cu at (171.7, 81.5)
Other:
- board text added: "LARA Proyect Lucas Herrera UPM 2026"
- board text added: "Status"

Commit message: pcb
Routing:
- net +12V: track 38.7 -> 38.0 mm
Changed lines of the file:
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@@
 	)
 	(segment
-		(start 171.0436 124.0536)
-		(end 168.1734 126.9238)
-		(width 1)
-		(layer "F.Cu")
-		(net 38)
-	)
-	(segment
-		(start 168.1734 126.9238)
-		(end 151.4238 126.9238)
-		(width 1)
-		(layer "F.Cu")
-		(net 38)
-	)
-	(segment
-		(start 151.4238 126.9238)
+		(start 150.484 125.984)
 		(end 148.5 124)
 		(width 1)
@@
 	)
 	(segment
-		(start 171.0436 113.4964)
-		(end 171.54 113)
+		(start 169.1132 125.984)
+		(end 150.484 125.984)
+		(width 1)
+		(layer "F.Cu")
+		(net 38)
+	)
+	(segment
+		(start 171.54 113)
+		(end 171.0436 113.4964)
 		(width 1)
 		(layer "F.Cu")
@@
 	)
 	(segment
-		(start 171.0436 124.0536)
-		(end 171.0436 113.4964)
+		(start 171.0436 113.4964)
+		(end 171.0436 124.0536)
 		(width 1)
 		(layer "F.Cu")
+		(net 38)
+	)
+	(segment
+		(start 171.0436 124.0536)
+		(end 169.1132 125.984)
+		(width 1)
+		(layer "F.Cu")
