File: pcb/LARA_hat/LARA_hat.kicad_sch (KiCad schematic)
At the start: 7 parts, among them J1 Raspberry_Pi_4, U1 MCP2515-xSO, U2 SN65HVD230, Y1 8MHz

Commit message: pcb
Parts:
- added J2: Conn_RoboClaw, Connector_JST:JST_PH_B3B-PH-K_1x03_P2.00mm_Vertical, symbol Connector:Conn_01x03_Pin
Changed lines of the file:
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@@
+	)
+	(symbol
+		(lib_id "Connector:Conn_01x03_Pin")
+		(at 34.29 63.5 0)
+		(unit 1)
+		(exclude_from_sim no)
+		(in_bom yes)
+		(on_board yes)
+		(dnp no)
+		(fields_autoplaced yes)
+		(property "Reference" "J2"
+			(at 34.925 55.88 0)
+			(effects
+				(font
+					(size 1.27 1.27)
+				)
+			)
+		)
+		(property "Value" "Conn_RoboClaw"
+			(at 34.925 58.42 0)
+			(effects
+				(font
+					(size 1.27 1.27)
+				)
+			)
+		)
+		(property "Footprint" "Connector_JST:JST_PH_B3B-PH-K_1x03_P2.00mm_Vertical"
+			(at 34.29 63.5 0)
+			(effects
+				(font
+					(size 1.27 1.27)
+				)
+				(hide yes)
+			)
+		)
+		(property "Datasheet" "~"
+			(at 34.29 63.5 0)
+			(effects
+				(font
+					(size 1.27 1.27)
+				)
+				(hide yes)
+			)
+		)
+		(property "Description" "Generic connector, single row, 01x03, script generated"
+			(at 34.29 63.5 0)
+			(effects
+				(font
+					(size 1.27 1.27)
+				)
+				(hide yes)
+			)
+		)
+		(pin "3"
+		)
+		(pin "2"
+		)
+		(pin "1"
+		)
+		(instances
+			(project ""
+				(path "/439a50f9-54cc-4d05-be8a-2234828ed849"
+					(reference "J2")
+					(unit 1)
+				)
+			)
+		)
 	)
 	(symbol

Commit message: pcb
Parts:
- added C3: 0.1u, symbol Device:C
- added J3: Conn_Dynamixel, Connector_JST:JST_EH_B3B-EH-A_1x03_P2.50mm_Vertical, symbol Connector:Conn_01x03_Pin
- added J4: Conn_01x02_Pin, symbol Connector:Conn_01x02_Pin
- added Q1, Q2, Q3: BSS138, Package_TO_SOT_SMD:SOT-23, symbol Transistor_FET:BSS138
- added R10, R2, R3, R4, R5, R6, R7, R8, R9: 10k, symbol Device:R
- added U3: 74LVC2G241, symbol 74xGxx:74LVC2G241
Connections:
- net +3V3: now also Q1.1 (G), Q2.1 (G), Q3.1 (G), R5.1, R7.1, R9.1
- net GND: now also C3.2, J3.1 (Pin_1), R4.2, U3.4 (GND)
- net at U2.6 (CANL): now also J4.2 (Pin_2)
- net at U2.7 (CANH): now also J4.1 (Pin_1)
- net at J1.13 (GPIO27/SDIO_DAT3): now also Q3.2 (S), R9.2
- net +5V: now reaches J1.2 (5V), J1.4 (5V)
- net +5V: now also C3.1, R10.1, R2.2, R3.1, R6.1, R8.1, U3.8 (VCC)
- net at J1.29 (GPCLK1/GPIO05): now also Q2.2 (S), R7.2
- net at J1.7 (GPCLK0/GPIO04): now also Q1.2 (S), R5.2
- new net: J3.3 (Pin_3), R2.1, U3.2, U3.3
- new net: Q2.3 (D), R3.2, R8.2, U3.6
- new net: Q1.3 (D), R6.2, U3.5
- new net: Q3.3 (D), R10.2, R4.1, U3.1, U3.7

Commit message: pcb update
Parts:
- removed Q1, Q2, Q3: BSS138, Package_TO_SOT_SMD:SOT-23, symbol Transistor_FET:BSS138
- removed R10, R5, R6, R7, R8, R9: 10k, symbol Device:R
- added C4: 1u, symbol Device:C
Connections:
- net +3V3: now also C3.1, R2.2, R3.1, U3.8 (VCC), C4.1
- net +5V: no longer C3.1, R2.2, R3.1, U3.8 (VCC)
- net GND: now also J1.13 (GPIO27/SDIO_DAT3), R4.1, U3.1, U3.7, C4.2
- net at J1.29 (GPCLK1/GPIO05): now also R3.2, U3.6
- net at U3.5: now also J1.7 (GPCLK0/GPIO04)
Other:
- moved on the sheet: C3, J3, R2, R3, R4, U3A, U3B, U3C

Commit message: pcb
Parts:
- added J5: 12V in, TerminalBlock:TerminalBlock_MaiXu_MX126-5.0-02P_1x02_P5.00mm, symbol Connector:Screw_Terminal_01x02
- added U4: ~, symbol components:BUCK12-5
- U3: footprint (none) -> Package_SO:VSSOP-8_3x3mm_P0.65mm
Connections:
- net +5V: now also U4.4 (5V_out)
- net GND: now also J2.3 (Pin_3), J5.2 (Pin_2), U4.2 (GND_in), U4.3 (GND_out); no longer J1.13 (GPIO27/SDIO_DAT3), R4.1, U3.1, U3.7
- net +12V: now reaches J3.2 (Pin_2)
- net +12V: now also J5.1 (Pin_1), U4.1 (12V_in)
- net at J2.1 (Pin_1): now also J1.8 (GPIO14/UART_TXD)
- net at J2.2 (Pin_2): now also J1.10 (GPIO15/UART_RXD)
- new net: J1.13 (GPIO27/SDIO_DAT3), R4.1, U3.1, U3.7

Commit message: pcb
Parts:
- C1, C2, C3: footprint (none) -> Capacitor_SMD:C_0805_2012Metric_Pad1.18x1.45mm_HandSolder
- R1, R2, R3, R4: footprint (none) -> Resistor_SMD:R_0805_2012Metric_Pad1.20x1.40mm_HandSolder
- U4: value ~ -> Buck 12V - 5V; footprint (none) -> components:BUCK12-5
Changed lines of the file:
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@@
 			)
 		)
-		(property "Footprint" ""
+		(property "Footprint" "Resistor_SMD:R_0805_2012Metric_Pad1.20x1.40mm_HandSolder"
 			(at 192.278 52.07 90)
 			(effects
@@
 			)
 		)
-		(property "Footprint" ""
+		(property "Footprint" "Capacitor_SMD:C_0805_2012Metric_Pad1.18x1.45mm_HandSolder"
 			(at 234.6452 43.18 0)
 			(effects
@@
 			)
 		)
-		(property "Footprint" ""
+		(property "Footprint" "Capacitor_SMD:C_0805_2012Metric_Pad1.18x1.45mm_HandSolder"
 			(at 50.8 147.6248 0)
 			(effects
@@
 			)
 		)
-		(property "Footprint" ""
+		(property "Footprint" "Resistor_SMD:R_0805_2012Metric_Pad1.20x1.40mm_HandSolder"
 			(at 155.702 52.07 90)
 			(effects
@@
 			)
 		)
-		(property "Footprint" ""
+		(property "Footprint" "Capacitor_SMD:C_0805_2012Metric_Pad1.18x1.45mm_HandSolder"
 			(at 50.8 159.0548 0)
 			(effects
@@
 			)
 		)
-		(property "Footprint" ""
+		(property "Footprint" "Resistor_SMD:R_0805_2012Metric_Pad1.20x1.40mm_HandSolder"
 			(at 109.982 156.21 90)
 			(effects
@@
 			)
 		)
-		(property "Value" "~"
+		(property "Value" "Buck 12V - 5V"
 			(at 80.01 27.94 0)
 			(effects
@@
 			)
 		)
-		(property "Footprint" ""
+		(property "Footprint" "components:BUCK12-5"
 			(at 80.01 29.21 0)
 			(effects
@@
 			)
 		)
-		(property "Footprint" ""
+		(property "Footprint" "Resistor_SMD:R_0805_2012Metric_Pad1.20x1.40mm_HandSolder"
 			(at 155.702 74.93 90)
 			(effects

Commit message: pcb
Parts:
- added D1: Rx_LED, LED_SMD:LED_0805_2012Metric_Pad1.15x1.40mm_HandSolder, symbol Device:LED
- added D2: Tx_LED, LED_SMD:LED_0805_2012Metric_Pad1.15x1.40mm_HandSolder, symbol Device:LED
- added D3: S0, LED_SMD:LED_0805_2012Metric_Pad1.15x1.40mm_HandSolder, symbol Device:LED
- added D4: S1, LED_SMD:LED_0805_2012Metric_Pad1.15x1.40mm_HandSolder, symbol Device:LED
- added D5: S2, LED_SMD:LED_0805_2012Metric_Pad1.15x1.40mm_HandSolder, symbol Device:LED
- added J7: I2C_JST, Connector_JST:JST_PH_B4B-PH-K_1x04_P2.00mm_Vertical, symbol Connector:Conn_01x04_Pin
- added R10, R6, R7, R8, R9: 68, Resistor_SMD:R_0805_2012Metric_Pad1.20x1.40mm_HandSolder, symbol Device:R
- added R5: 120, Resistor_SMD:R_0805_2012Metric_Pad1.20x1.40mm_HandSolder, symbol Device:R
- C4: footprint (none) -> Capacitor_SMD:C_0805_2012Metric_Pad1.18x1.45mm_HandSolder
- J4: footprint (none) -> Connector_JST:JST_PH_B2B-PH-K_1x02_P2.00mm_Vertical
- Y1: footprint (none) -> Crystal:Crystal_HC49-4H_Vertical
Connections:
- net +3V3: now also J7.1 (Pin_1)
- net GND: now also J7.2 (Pin_2), R10.2, R6.2, R7.2, R8.2, R9.2
- net at J4.1 (Pin_1), U2.7 (CANH): now also R5.1
- net at J4.2 (Pin_2), U2.6 (CANL): now also R5.2
- net at U1.1 (TXCAN), U2.1 (D): now also D1.2 (A)
- net at U1.2 (RXCAN), U2.4 (R): now also D2.2 (A)
- net at J1.15 (GPIO22/SDIO_CLK): now also D3.2 (A)
- net at J1.16 (GPIO23/SDIO_CMD): now also D4.2 (A)
- net at J1.18 (GPIO24/SDIO_DAT0): now also D5.2 (A)
- net at J1.3 (SDA_I2C1/GPIO02): now also J7.3 (Pin_3)
- net at J1.5 (SCL_I2C1/GPIO03): now also J7.4 (Pin_4)
- new net: D4.1 (K), R9.1
- new net: D3.1 (K), R8.1
- new net: D1.1 (K), R6.1
- new net: D2.1 (K), R7.1
- new net: D5.1 (K), R10.1
Other:
- moved on the sheet: J4, R1, U2

Commit message: pcb
Parts:
- added J6: LED_JST, Connector_JST:JST_PH_B4B-PH-K_1x04_P2.00mm_Vertical, symbol Connector:Conn_01x04_Pin
Connections:
- net GND: now also J6.4 (Pin_4)
- net at D4.2 (A), J1.16 (GPIO23/SDIO_CMD): now also J6.2 (Pin_2)
- net at D3.2 (A), J1.15 (GPIO22/SDIO_CLK): now also J6.1 (Pin_1)
- net at D5.2 (A), J1.18 (GPIO24/SDIO_DAT0): now also J6.3 (Pin_3)

Commit message: pcb
Parts:
- R10, R8, R9: value 68 -> 47
Changed lines of the file:
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@@
 			)
 		)
-		(property "Value" "68"
+		(property "Value" "47"
 			(at 25.4 106.6799 0)
 			(effects
@@
 			)
 		)
-		(property "Value" "68"
+		(property "Value" "47"
 			(at 34.29 109.2199 0)
 			(effects
@@
 			)
 		)
-		(property "Value" "68"
+		(property "Value" "47"
 			(at 43.18 111.7599 0)
 			(effects
