File: pcb/intercons2/intercons2.kicad_pcb (KiCad board)
At the start: 2 copper layers, 77.8 x 84.6 mm, 15 parts, among them J1 PSU, J2 BATTERY, J3 Raspberry, J4 RoboClaw1, J5 RoboClaw2, SW1 PWR_SWITCH

Commit message: pcb
Other:
- board text added: "Raspberry"
- board text removed: "PSU"
Changed lines of the file:
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@@
 		(tenting front back)
 		(pcbplotparams
-			(layerselection 0x00000000_00000000_5555555f_575555ff)
+			(layerselection 0x00000000_00000000_5555555f_5755f5ff)
 			(plot_on_all_layers_selection 0x00000000_00000000_00000000_00000000)
 			(disableapertmacros no)
-			(usegerberextensions no)
+			(usegerberextensions yes)
 			(usegerberattributes yes)
 			(usegerberadvancedattributes yes)
-			(creategerberjobfile yes)
+			(creategerberjobfile no)
 			(dashed_line_dash_ratio 12.000000)
 			(dashed_line_gap_ratio 3.000000)
@@
 		)
 		(property "Value" "BATTERY"
-			(at 2.286 6.0452 90)
+			(at 2.146 6.196 90)
 			(layer "F.Fab")
 			(effects
@@
 		)
 	)
+	(gr_text "Raspberry"
+		(at 109 66 90)
+		(layer "F.SilkS")
+		(effects
+			(font
+				(size 1 1)
+				(thickness 0.15)
+			)
+		)
+	)
 	(gr_text "RoboClaw2"
-		(at 109.8296 104.5718 90)
+		(at 110 113.5 90)
 		(layer "F.SilkS")
 		(effects
@@
 	)
 	(gr_text "BATTERY"
-		(at 165.2524 119.4816 90)
+		(at 165 104 90)
 		(layer "F.SilkS")
 		(effects
@@
 		)
 	)
-	(gr_text "PSU"
-		(at 165.7604 104.7496 90)
-		(layer "F.Fab")
-		(effects
-			(font
-				(size 1 1)
-				(thickness 0.15)
-			)
-		)
-	)
 	(segment
 		(start 156.3044 111.9124)
@@
 	)
 	(segment
-		(start 138.1506 96.6216)
-		(end 138.1506 93.5482)
-		(width 2)
-		(layer "F.Cu")
-		(net 2)
-	)
-	(segment
-		(start 118.3885 73.7861)
-		(end 118.3885 69.9301)
-		(width 2)
-		(layer "F.Cu")
-		(net 2)
-	)
-	(segment
-		(start 138.1506 93.5482)
-		(end 118.3885 73.7861)
+		(start 120.5 76.5)
+		(end 120.5 72.0416)
 		(width 2)
 		(layer "F.Cu")
@@
 	)
 	(segment
-		(start 118.3885 69.9301)
+		(start 131.4196 103.3526)
+		(end 138.1506 96.6216)
+		(width 2)
+		(layer "F.Cu")
+		(net 2)
+	)
+	(segment
+		(start 120.5 72.0416)
 		(end 116.235 67.7766)
 		(width 2)
@@
 	)
 	(segment
-		(start 131.4196 103.3526)
-		(end 138.1506 96.6216)
+		(start 138.1506 96.6216)
+		(end 138.1506 94.1506)
 		(width 2)
 		(layer "F.Cu")
@@
 		(width 2)
 		(layer "F.Cu")
+		(net 2)
+	)
+	(segment
+		(start 138.1506 94.1506)
+		(end 120.5 76.5)
+		(width 2)
+		(layer "F.Cu")
